Commit message: localization correction

File: src/hightorque_robot/Panthera-HT_description/urdf/Panthera-HT_description_follower.urdf (robot description, URDF)
Before this commit: robot Panthera-HT_description, 7 links, 6 joints
Links:
- added link gripper_center
Joints:
- added joint gripper_center_joint: type fixed, parent link6, child gripper_center, origin xyz=0.1701 0 0 rpy=0 0 0

File: src/panthera_ht_description_with_finger/urdf/Panthera-HT_description_with_finger.urdf (robot description, URDF)
Before this commit: robot Panthera-HT_description, 9 links, 8 joints
Links:
- added link gripper_center
Joints:
- added joint gripper_center_joint: type fixed, parent link6, child gripper_center, origin xyz=0.1701 0 0 rpy=0 0 0
- joint L_finger: origin xyz=0.16555 0 0 rpy=0 0 0 -> xyz=-0.00455 0 0 rpy=0 0 0; parent link6 -> gripper_center
- joint R_finger: origin xyz=0.16555 0 0 rpy=0 0 0 -> xyz=-0.00455 0 0 rpy=0 0 0; parent link6 -> gripper_center

File: src/panthera_ht_description_with_finger/urdf/Panthera-HT_description_with_finger.urdf.xacro (robot description, xacro)
@@ -202,4 +202,11 @@
     <dynamics damping="0.7" friction="0.0"/>
   </joint>
+  <!-- Tool center point at the center of the gripper fingertips. -->
+  <link name="gripper_center" />
+  <joint name="gripper_center_joint" type="fixed">
+    <origin xyz="0.1701 0 0" rpy="0 0 0" />
+    <parent link="link6" />
+    <child link="gripper_center" />
+  </joint>
   <link name="L_finger">
     <inertial>
@@ -224,6 +231,6 @@
   </link>
   <joint name="L_finger_joint" type="prismatic">
-    <origin xyz="0.16555 0 0" rpy="0 0 0" />
-    <parent link="link6" />
+    <origin xyz="-0.00455 0 0" rpy="0 0 0" />
+    <parent link="gripper_center" />
     <child link="L_finger" />
     <axis xyz="0 1 0" />
@@ -253,6 +260,6 @@
   </link>
   <joint name="R_finger_joint" type="prismatic">
-    <origin xyz="0.16555 0 0" rpy="0 0 0" />
-    <parent link="link6" />
+    <origin xyz="-0.00455 0 0" rpy="0 0 0" />
+    <parent link="gripper_center" />
     <child link="R_finger" />
     <axis xyz="0 -1 0" />
