Commit message: 更新Lyrical适配

File: src/panthera_gazebo/urdf/gazebo.xacro (robot description, xacro)
@@ -94,4 +94,8 @@
       <robot_param_node>robot_state_publisher</robot_param_node>
       <parameters>$(arg ros2_control_params)</parameters>
+      <!-- The upstream default (0.1) leaves roughly 0.1 rad of tracking lag
+           on this model's fastest trajectories. A unit gain tracks each
+           controller update without relaxing trajectory tolerances. -->
+      <position_proportional_gain>1.0</position_proportional_gain>
     </plugin>
   </gazebo>

File: src/panthera_ht_config/config/panthera_ht_hardware.ros2_control.xacro (robot description, xacro)
@@ -13,4 +13,6 @@
             <joint name="joint1">
                 <command_interface name="position"/>
+                <command_interface name="velocity"/>
+                <command_interface name="effort"/>
                 <state_interface name="position"/>
                 <state_interface name="velocity"/>
@@ -24,4 +26,6 @@
             <joint name="joint2">
                 <command_interface name="position"/>
+                <command_interface name="velocity"/>
+                <command_interface name="effort"/>
                 <state_interface name="position"/>
                 <state_interface name="velocity"/>
@@ -35,4 +39,6 @@
             <joint name="joint3">
                 <command_interface name="position"/>
+                <command_interface name="velocity"/>
+                <command_interface name="effort"/>
                 <state_interface name="position"/>
                 <state_interface name="velocity"/>
@@ -46,4 +52,6 @@
             <joint name="joint4">
                 <command_interface name="position"/>
+                <command_interface name="velocity"/>
+                <command_interface name="effort"/>
                 <state_interface name="position"/>
                 <state_interface name="velocity"/>
@@ -57,4 +65,6 @@
             <joint name="joint5">
                 <command_interface name="position"/>
+                <command_interface name="velocity"/>
+                <command_interface name="effort"/>
                 <state_interface name="position"/>
                 <state_interface name="velocity"/>
@@ -68,4 +78,6 @@
             <joint name="joint6">
                 <command_interface name="position"/>
+                <command_interface name="velocity"/>
+                <command_interface name="effort"/>
                 <state_interface name="position"/>
                 <state_interface name="velocity"/>

File: src/panthera_ht_config/config/panthera_ht_ros_description.ros2_control.xacro (robot description, xacro)
@@ -1,5 +1,6 @@
 <?xml version="1.0"?>
 <robot xmlns:xacro="http://www.ros.org/wiki/xacro">
-    <xacro:macro name="panthera_ht_ros_description_ros2_control" params="name initial_positions_file use_mock_hardware:=true">
+    <xacro:macro name="panthera_ht_ros_description_ros2_control"
+                 params="name initial_positions_file use_mock_hardware:=true config_file control_mode">
         <xacro:property name="initial_positions" value="${xacro.load_yaml(initial_positions_file)['initial_positions']}"/>
         <ros2_control name="${name}" type="system">
@@ -10,11 +11,13 @@
                 </xacro:if>
                 <xacro:unless value="${use_mock_hardware}">
-                    <!-- 真实硬件 - 使用 Panthera Python SDK -->
-                    <plugin>panthera_hardware/PantheraSystemHardware</plugin>
-                    <param name="config_path">/home/hightorque/Panthera-HT_ros2_ws/src/panthera_python/robot_param/Leader.yaml</param>
+                    <plugin>panthera_hardware/PantheraHardwareInterface</plugin>
+                    <param name="config_file">${config_file}</param>
+                    <param name="control_mode">${control_mode}</param>
                 </xacro:unless>
             </hardware>
             <joint name="joint1">
                 <command_interface name="position"/>
+                <command_interface name="velocity"/>
+                <command_interface name="effort"/>
                 <state_interface name="position">
                   <param name="initial_value">${initial_positions['joint1']}</param>
@@ -25,4 +28,6 @@
             <joint name="joint2">
                 <command_interface name="position"/>
+                <command_interface name="velocity"/>
+                <command_interface name="effort"/>
                 <state_interface name="position">
                   <param name="initial_value">${initial_positions['joint2']}</param>
@@ -33,4 +38,6 @@
             <joint name="joint3">
                 <command_interface name="position"/>
+                <command_interface name="velocity"/>
+                <command_interface name="effort"/>
                 <state_interface name="position">
                   <param name="initial_value">${initial_positions['joint3']}</param>
@@ -41,4 +48,6 @@
             <joint name="joint4">
                 <command_interface name="position"/>
+                <command_interface name="velocity"/>
+                <command_interface name="effort"/>
                 <state_interface name="position">
                   <param name="initial_value">${initial_positions['joint4']}</param>
@@ -49,4 +58,6 @@
             <joint name="joint5">
                 <command_interface name="position"/>
+                <command_interface name="velocity"/>
+                <command_interface name="effort"/>
                 <state_interface name="position">
                   <param name="initial_value">${initial_positions['joint5']}</param>
@@ -57,4 +68,6 @@
             <joint name="joint6">
                 <command_interface name="position"/>
+                <command_interface name="velocity"/>
+                <command_interface name="effort"/>
                 <state_interface name="position">
                   <param name="initial_value">${initial_positions['joint6']}</param>

File: src/panthera_ht_config/config/panthera_ht_ros_description.urdf.xacro (robot description, xacro)
@@ -3,4 +3,6 @@
     <xacro:arg name="initial_positions_file" default="initial_positions.yaml" />
     <xacro:arg name="use_mock_hardware" default="true" />
+    <xacro:arg name="config_file" default="$(find hightorque_robot)/robot_param/Follower_absolute.yaml" />
+    <xacro:arg name="control_mode" default="pd_control" />
     <!-- Import panthera_ht_ros_description urdf file -->
     <xacro:include filename="$(find panthera_ht_ros_description)/urdf/panthera_ht_ros_description.xacro" />
@@ -10,4 +12,6 @@
         name="FakeSystem"
         initial_positions_file="$(arg initial_positions_file)"
-        use_mock_hardware="$(arg use_mock_hardware)"/>
+        use_mock_hardware="$(arg use_mock_hardware)"
+        config_file="$(arg config_file)"
+        control_mode="$(arg control_mode)"/>
 </robot>

File: src/panthera_ht_ros_description/urdf/panthera_ht_ros_description_gripper.urdf.xacro (robot description, xacro)
@@ -14,4 +14,5 @@
       <command_interface name="position"/>
       <command_interface name="velocity"/>
+      <command_interface name="effort"/>
       <state_interface name="position"/>
       <state_interface name="velocity"/>
@@ -25,4 +26,5 @@
       <command_interface name="position"/>
       <command_interface name="velocity"/>
+      <command_interface name="effort"/>
       <state_interface name="position"/>
       <state_interface name="velocity"/>
@@ -36,4 +38,5 @@
       <command_interface name="position"/>
       <command_interface name="velocity"/>
+      <command_interface name="effort"/>
       <state_interface name="position"/>
       <state_interface name="velocity"/>
@@ -47,4 +50,5 @@
       <command_interface name="position"/>
       <command_interface name="velocity"/>
+      <command_interface name="effort"/>
       <state_interface name="position"/>
       <state_interface name="velocity"/>
@@ -58,4 +62,5 @@
       <command_interface name="position"/>
       <command_interface name="velocity"/>
+      <command_interface name="effort"/>
       <state_interface name="position"/>
       <state_interface name="velocity"/>
@@ -69,4 +74,5 @@
       <command_interface name="position"/>
       <command_interface name="velocity"/>
+      <command_interface name="effort"/>
       <state_interface name="position"/>
       <state_interface name="velocity"/>
@@ -80,4 +86,5 @@
       <command_interface name="position"/>
       <command_interface name="velocity"/>
+      <command_interface name="effort"/>
       <state_interface name="position"/>
       <state_interface name="velocity"/>

File: src/panthera_ht_ros_description/urdf/panthera_ht_ros_description_gripper.xacro (robot description, xacro)
@@ -1,4 +1,25 @@
 <?xml version="1.0"?>
 <robot xmlns:xacro="http://www.ros.org/wiki/xacro" name="panthera_ht_ros_description">
+  <!-- Keep the detailed STL collision model for MoveIt, while allowing
+       physics simulators to request inexpensive primitive collisions. -->
+  <xacro:arg name="use_mesh_collisions" default="true"/>
+  <xacro:macro name="panthera_collision" params="mesh_name box_origin box_size">
+    <xacro:if value="$(arg use_mesh_collisions)">
+      <collision>
+        <origin xyz="0 0 0" rpy="0 0 0"/>
+        <geometry>
+          <mesh filename="package://panthera_ht_ros_description/meshes/${mesh_name}.STL"/>
+        </geometry>
+      </collision>
+    </xacro:if>
+    <xacro:unless value="$(arg use_mesh_collisions)">
+      <collision>
+        <origin xyz="${box_origin}" rpy="0 0 0"/>
+        <geometry>
+          <box size="${box_size}"/>
+        </geometry>
+      </collision>
+    </xacro:unless>
+  </xacro:macro>
   <mujoco>
     <compiler meshdir="../meshes/" balanceinertia="true" discardvisual="false"/>
@@ -15,8 +36,6 @@
       <material name=""><color rgba="0.752941176470588 0.752941176470588 0.752941176470588 1"/></material>
     </visual>
-    <collision>
-      <origin xyz="0 0 0" rpy="0 0 0"/>
-      <geometry><mesh filename="package://panthera_ht_ros_description/meshes/base_link.STL"/></geometry>
-    </collision>
+    <xacro:panthera_collision mesh_name="base_link"
+      box_origin="0 0 0.03035" box_size="0.12 0.12 0.0607"/>
   </link>
   <link name="link1">
@@ -31,8 +50,6 @@
       <material name=""><color rgba="0.752941176470588 0.752941176470588 0.752941176470588 1"/></material>
     </visual>
-    <collision>
-      <origin xyz="0 0 0" rpy="0 0 0"/>
-      <geometry><mesh filename="package://panthera_ht_ros_description/meshes/link1.STL"/></geometry>
-    </collision>
+    <xacro:panthera_collision mesh_name="link1"
+      box_origin="0.005815505 0 0.03825" box_size="0.071631039 0.087 0.0765"/>
   </link>
   <joint name="joint1" type="revolute">
@@ -54,8 +71,7 @@
       <material name=""><color rgba="0.752941176470588 0.752941176470588 0.752941176470588 1"/></material>
     </visual>
-    <collision>
-      <origin xyz="0 0 0" rpy="0 0 0"/>
-      <geometry><mesh filename="package://panthera_ht_ros_description/meshes/link2.STL"/></geometry>
-    </collision>
+    <xacro:panthera_collision mesh_name="link2"
+      box_origin="-0.130000004 0.000500001 0.002256604"
+      box_size="0.32200001 0.066500001 0.066513207"/>
   </link>
   <joint name="joint2" type="revolute">
@@ -77,8 +93,7 @@
       <material name=""><color rgba="0.752941176470588 0.752941176470588 0.752941176470588 1"/></material>
     </visual>
-    <collision>
-      <origin xyz="0 0 0" rpy="0 0 0"/>
-      <geometry><mesh filename="package://panthera_ht_ros_description/meshes/link3.STL"/></geometry>
-    </collision>
+    <xacro:panthera_collision mesh_name="link3"
+      box_origin="0.116249999 0 0.031251292"
+      box_size="0.279500026 0.080499999 0.109497422"/>
   </link>
   <joint name="joint3" type="revolute">
@@ -100,8 +115,7 @@
       <material name=""><color rgba="0.752941176470588 0.752941176470588 0.752941176470588 1"/></material>
     </visual>
-    <collision>
-      <origin xyz="0 0 0" rpy="0 0 0"/>
-      <geometry><mesh filename="package://panthera_ht_ros_description/meshes/link4.STL"/></geometry>
-    </collision>
+    <xacro:panthera_collision mesh_name="link4"
+      box_origin="0.036006011 0.000000864 0.029863416"
+      box_size="0.111987978 0.075638272 0.09971145"/>
   </link>
   <joint name="joint4" type="revolute">
@@ -123,8 +137,6 @@
       <material name=""><color rgba="0.752941176470588 0.752941176470588 0.752941176470588 1"/></material>
     </visual>
-    <collision>
-      <origin xyz="0 0 0" rpy="0 0 0"/>
-      <geometry><mesh filename="package://panthera_ht_ros_description/meshes/link5.STL"/></geometry>
-    </collision>
+    <xacro:panthera_collision mesh_name="link5"
+      box_origin="0.001 0 -0.035572179" box_size="0.0519 0.044 0.071144358"/>
   </link>
   <joint name="joint5" type="revolute">
@@ -146,8 +158,6 @@
       <material name=""><color rgba="0.752941176470588 0.752941176470588 0.752941176470588 1"/></material>
     </visual>
-    <collision>
-      <origin xyz="0 0 0" rpy="0 0 0"/>
-      <geometry><mesh filename="package://panthera_ht_ros_description/meshes/link6.STL"/></geometry>
-    </collision>
+    <xacro:panthera_collision mesh_name="link6"
+      box_origin="0.0055 0 0.003" box_size="0.011 0.03 0.036"/>
   </link>
   <joint name="joint6" type="revolute">
@@ -169,8 +179,6 @@
       <material name=""><color rgba="0.752941176470588 0.752941176470588 0.752941176470588 1"/></material>
     </visual>
-    <collision>
-      <origin xyz="0 0 0" rpy="0 0 0"/>
-      <geometry><mesh filename="package://panthera_ht_ros_description/meshes/L_finger.STL"/></geometry>
-    </collision>
+    <xacro:panthera_collision mesh_name="L_finger"
+      box_origin="-0.047424598 0.0175 0" box_size="0.105050805 0.035 0.041"/>
   </link>
   <joint name="L_finger_joint" type="prismatic">
@@ -192,8 +200,6 @@
       <material name=""><color rgba="0.752941176470588 0.752941176470588 0.752941176470588 1"/></material>
     </visual>
-    <collision>
-      <origin xyz="0 0 0" rpy="0 0 0"/>
-      <geometry><mesh filename="package://panthera_ht_ros_description/meshes/R_finger.STL"/></geometry>
-    </collision>
+    <xacro:panthera_collision mesh_name="R_finger"
+      box_origin="-0.047424598 -0.0175 0" box_size="0.105050805 0.035 0.041"/>
   </link>
   <joint name="R_finger_joint" type="prismatic">
@@ -216,8 +222,6 @@
       <material name=""><color rgba="0.866666666666667 0.909803921568627 1 1"/></material>
     </visual>
-    <collision>
-      <origin xyz="0 0 0" rpy="0 0 0"/>
-      <geometry><mesh filename="package://panthera_ht_ros_description/meshes/gripper_center.STL"/></geometry>
-    </collision>
+    <xacro:panthera_collision mesh_name="gripper_center"
+      box_origin="-0.124950003 0 0" box_size="0.072000004 0.158000007 0.037"/>
   </link>
   <joint name="gripper_center_joint" type="fixed">

File: src/panthera_ht_ros_description/urdf/panthera_ht_ros_description_hardware.urdf.xacro (robot description, xacro)
@@ -4,7 +4,7 @@
   <xacro:include filename="$(find panthera_ht_ros_description)/urdf/panthera_ht_ros_description.xacro"/>
   <!-- Include the hardware ros2_control configuration -->
-  <xacro:include filename="$(find panthera-ht_hardware)/config/panthera_hardware.ros2_control.xacro"/>
+  <xacro:include filename="$(find panthera_hardware)/config/panthera_hardware.ros2_control.xacro"/>
   <!-- Parameters -->
-  <xacro:arg name="config_file" default="$(find panthera_robot)/robot_param/Leader.yaml"/>
+  <xacro:arg name="config_file" default="$(find hightorque_robot)/robot_param/Follower_absolute.yaml"/>
   <xacro:arg name="control_mode" default="position_velocity"/>
   <!-- Instantiate the hardware ros2_control -->
