Commit message: Organize the file structure

File: src/hightorque_robot/urdf/Panthera-HT_description_follower.urdf (robot description, URDF)
Before this commit: robot Panthera-HT_description, 8 links, 7 joints
Links:
- link base_link: geometry collision mesh filename=package://panthera_ht_description/meshes/base_link.STL; visual mesh filename=package://panthera_ht_description/meshes/base_link.STL
- link link1: geometry collision mesh filename=package://panthera_ht_description/meshes/link1.STL; visual mesh filename=package://panthera_ht_description/meshes/link1.STL
- link link2: geometry collision mesh filename=package://panthera_ht_description/meshes/link2.STL; visual mesh filename=package://panthera_ht_description/meshes/link2.STL
- link link3: geometry collision mesh filename=package://panthera_ht_description/meshes/link3.STL; visual mesh filename=package://panthera_ht_description/meshes/link3.STL
- link link4: geometry collision mesh filename=package://panthera_ht_description/meshes/link4.STL; visual mesh filename=package://panthera_ht_description/meshes/link4.STL
- link link5: geometry collision mesh filename=package://panthera_ht_description/meshes/link5.STL; visual mesh filename=package://panthera_ht_description/meshes/link5.STL
- link link6: geometry collision mesh filename=package://panthera_ht_description/meshes/link6.STL; visual mesh filename=package://panthera_ht_description/meshes/link6.STL

File: src/panthera_gazebo/urdf/Panthera-HT_gazebo.urdf.xacro (robot description, xacro)
@@ -1,10 +1,10 @@
 <?xml version="1.0"?>
-<robot xmlns:xacro="http://www.ros.org/wiki/xacro" name="Panthera-HT_description">
+<robot xmlns:xacro="http://www.ros.org/wiki/xacro" name="panthera_ht_ros_description">
     <xacro:arg name="initial_positions_file"
-               default="$(find with_gripper_config)/config/initial_positions.yaml" />
+               default="$(find panthera_moveit_config)/config/initial_positions.yaml" />
     <xacro:arg name="ros2_control_params"
                default="$(find panthera_gazebo)/config/ros2_controllers.yaml" />
     <!-- 1. Import base URDF -->
-    <xacro:include filename="$(find panthera_ht_description_with_finger)/urdf/Panthera-HT_description_with_finger.urdf.xacro" />
+    <xacro:include filename="$(find panthera_ht_description)/urdf/panthera_ht_ros_description_gripper.urdf.xacro" />
     <!-- 2. Import Gazebo configuration (materials, friction, world joint, plugin) -->
     <xacro:include filename="$(find panthera_gazebo)/urdf/gazebo.xacro" />

File: src/panthera_gazebo/urdf/Panthera-HT_gazebo_classic.urdf.xacro (robot description, xacro)
@@ -1,10 +1,10 @@
 <?xml version="1.0"?>
-<robot xmlns:xacro="http://www.ros.org/wiki/xacro" name="Panthera-HT_description">
+<robot xmlns:xacro="http://www.ros.org/wiki/xacro" name="panthera_ht_ros_description">
     <xacro:arg name="initial_positions_file"
-               default="$(find with_gripper_config)/config/initial_positions.yaml" />
+               default="$(find panthera_moveit_config)/config/initial_positions.yaml" />
     <xacro:arg name="ros2_control_params"
                default="$(find panthera_gazebo)/config/ros2_controllers.yaml" />
     <!-- 1. Import base URDF -->
-    <xacro:include filename="$(find panthera_ht_description_with_finger)/urdf/Panthera-HT_description_with_finger.urdf.xacro" />
+    <xacro:include filename="$(find panthera_ht_description)/urdf/panthera_ht_ros_description_gripper.urdf.xacro" />
     <!-- 2. Import Gazebo Classic configuration -->
     <xacro:include filename="$(find panthera_gazebo)/urdf/gazebo_classic.xacro" />

File: src/panthera_ht_description/urdf/panthera_ht_ros_description_gripper.urdf (robot description, URDF)
Before this commit: robot Panthera-HT_description, 10 links, 9 joints
Links:
- link L_finger: geometry collision mesh filename=package://panthera_ht_description/meshes/L_finger.STL; visual mesh filename=package://panthera_ht_description/meshes/L_finger.STL
- link R_finger: geometry collision mesh filename=package://panthera_ht_description/meshes/R_finger.STL; visual mesh filename=package://panthera_ht_description/meshes/R_finger.STL
- link base_link: geometry collision mesh filename=package://panthera_ht_description/meshes/base_link.STL; visual mesh filename=package://panthera_ht_description/meshes/base_link.STL
- link link1: geometry collision mesh filename=package://panthera_ht_description/meshes/link1.STL; visual mesh filename=package://panthera_ht_description/meshes/link1.STL
- link link2: geometry collision mesh filename=package://panthera_ht_description/meshes/link2.STL; visual mesh filename=package://panthera_ht_description/meshes/link2.STL
- link link3: geometry collision mesh filename=package://panthera_ht_description/meshes/link3.STL; visual mesh filename=package://panthera_ht_description/meshes/link3.STL
- link link4: geometry collision mesh filename=package://panthera_ht_description/meshes/link4.STL; visual mesh filename=package://panthera_ht_description/meshes/link4.STL
- link link5: geometry collision mesh filename=package://panthera_ht_description/meshes/link5.STL; visual mesh filename=package://panthera_ht_description/meshes/link5.STL
- link link6: mass 0.45 -> 0.43; geometry collision mesh filename=package://panthera_ht_description/meshes/link6.STL; visual mesh filename=package://panthera_ht_description/meshes/link6.STL

File: src/panthera_ht_description/urdf/panthera_ht_ros_description_gripper.urdf.xacro (robot description, xacro)
@@ -3,7 +3,7 @@
      Commit Version: 1.6.0-4-g7f85cfe  Build Version: 1.6.7995.38578
      For more information, please see http://wiki.ros.org/sw_urdf_exporter -->
-<robot name="Panthera-HT_description" xmlns:xacro="http://www.ros.org/wiki/xacro">
+<robot name="panthera_ht_ros_description" xmlns:xacro="http://www.ros.org/wiki/xacro">
   <!-- Xacro properties for commonly used values -->
-  <xacro:property name="package_name" value="panthera_ht_description_with_finger" />
+  <xacro:property name="package_name" value="panthera_ht_description" />
   <xacro:property name="default_color" value="0.752941176470588 0.752941176470588 0.752941176470588 1" />
   <!-- Material definitions -->
@@ -177,5 +177,5 @@
     <inertial>
       <origin xyz="0.06704625 0.00051731 1.674e-05" rpy="0 0 0" />
-      <mass value="0.45" />
+      <mass value="0.43" />
       <inertia ixx="0.00107368" ixy="-1.25e-05" ixz="3e-07" iyy="0.00068998" iyz="2.517e-05" izz="0.00167551" />
     </inertial>
@@ -235,5 +235,5 @@
     <child link="L_finger" />
     <axis xyz="0 1 0" />
-    <limit lower="-5.0" upper="5.0" effort="100" velocity="0.5" />
+    <limit lower="0.0" upper="0.04" effort="100" velocity="0.1" />
     <dynamics damping="0.5" friction="0.0"/>
   </joint>
@@ -263,8 +263,8 @@
     <parent link="gripper_center" />
     <child link="R_finger" />
-    <axis xyz="0 -1 0" />
-    <limit lower="-5.0" upper="5.0" effort="100" velocity="0.5" />
+    <axis xyz="0 1 0" />
+    <limit lower="-0.04" upper="0.0" effort="100" velocity="0.1" />
     <dynamics damping="0.5" friction="0.0"/>
-    <mimic joint="L_finger_joint" multiplier="1" offset="0"/>
+    <mimic joint="L_finger_joint" multiplier="-1" offset="0"/>
   </joint>
 </robot>

File: src/panthera_moveit_config/config/panthera_ht_hardware.ros2_control.xacro (robot description, xacro)
@@ -1,5 +1,5 @@
 <?xml version="1.0"?>
 <robot xmlns:xacro="http://www.ros.org/wiki/xacro">
-    <xacro:macro name="Panthera-HT_description_hardware_ros2_control" params="name config_file control_mode">
+    <xacro:macro name="panthera_ht_ros_description_hardware_ros2_control" params="name config_file control_mode">
         <ros2_control name="${name}" type="system">
             <hardware>
@@ -8,5 +8,5 @@
                 <param name="config_file">${config_file}</param>
                 <param name="control_mode">${control_mode}</param>
-                <param name="gripper_rad_to_m">0.04</param>
+                <param name="gripper_rad_to_m">0.025</param>
             </hardware>
             <!-- Joint 1 -->

File: src/panthera_moveit_config/config/panthera_ht_hardware.urdf.xacro (robot description, xacro)
@@ -1,12 +1,12 @@
 <?xml version="1.0"?>
-<robot xmlns:xacro="http://www.ros.org/wiki/xacro" name="Panthera-HT_description">
+<robot xmlns:xacro="http://www.ros.org/wiki/xacro" name="panthera_ht_ros_description">
     <xacro:arg name="config_file" default="$(find hightorque_robot)/robot_param/Leader.yaml" />
     <xacro:arg name="control_mode" default="position_velocity" />
-    <!-- Import Panthera-HT_description urdf file -->
-    <xacro:include filename="$(find panthera_ht_description_with_finger)/urdf/Panthera-HT_description_with_finger.urdf.xacro" />
+    <!-- Import panthera_ht_ros_description urdf file -->
+    <xacro:include filename="$(find panthera_ht_description)/urdf/panthera_ht_ros_description_gripper.urdf.xacro" />
     <!-- Import hardware control_xacro -->
-    <xacro:include filename="Panthera-HT_description_hardware.ros2_control.xacro" />
+    <xacro:include filename="panthera_ht_hardware.ros2_control.xacro" />
     <!-- Instantiate hardware interface -->
-    <xacro:Panthera-HT_description_hardware_ros2_control
+    <xacro:panthera_ht_ros_description_hardware_ros2_control
         name="PantheraHardware"
         config_file="$(arg config_file)"

File: src/panthera_moveit_config/config/panthera_ht_ros_description.ros2_control.xacro (robot description, xacro)
@@ -1,5 +1,5 @@
 <?xml version="1.0"?>
 <robot xmlns:xacro="http://www.ros.org/wiki/xacro">
-    <xacro:macro name="Panthera-HT_description_ros2_control" params="name initial_positions_file">
+    <xacro:macro name="panthera_ht_ros_description_ros2_control" params="name initial_positions_file">
         <xacro:property name="initial_positions" value="${xacro.load_yaml(initial_positions_file)['initial_positions']}"/>
         <ros2_control name="${name}" type="system">

File: src/panthera_moveit_config/config/panthera_ht_ros_description.urdf.xacro (robot description, xacro)
@@ -1,9 +1,9 @@
 <?xml version="1.0"?>
-<robot xmlns:xacro="http://www.ros.org/wiki/xacro" name="Panthera-HT_description">
+<robot xmlns:xacro="http://www.ros.org/wiki/xacro" name="panthera_ht_ros_description">
     <xacro:arg name="initial_positions_file" default="initial_positions.yaml" />
-    <!-- Import Panthera-HT_description urdf file -->
-    <xacro:include filename="$(find panthera_ht_description_with_finger)/urdf/Panthera-HT_description_with_finger.urdf.xacro" />
+    <!-- Import panthera_ht_ros_description urdf file -->
+    <xacro:include filename="$(find panthera_ht_description)/urdf/panthera_ht_ros_description_gripper.urdf.xacro" />
     <!-- Import control_xacro -->
-    <xacro:include filename="Panthera-HT_description.ros2_control.xacro" />
-    <xacro:Panthera-HT_description_ros2_control name="FakeSystem" initial_positions_file="$(arg initial_positions_file)"/>
+    <xacro:include filename="panthera_ht_ros_description.ros2_control.xacro" />
+    <xacro:panthera_ht_ros_description_ros2_control name="FakeSystem" initial_positions_file="$(arg initial_positions_file)"/>
 </robot>
